File: vreg-741.kicad_pcb (KiCad board)
At the start: 2 copper layers, 46.2 x 24.9 mm, 24 parts, among them J1 1729128, J2 1729128, Q1 FQT5P10, Q2 2STN1550, SW1 A6SN-1104, U1 UA741CDR‎

Commit message: extra easter eggs
Parts:
- added G***: LOGO, marion:avengers, F.Cu at (201.9, 79.2)
- moved G*** 1.14 mm to (188.3, 78.7)
Other:
- board text added: "Ah we can dance if we want to, we can leave your friends behind. Cause your friends don't dance and if they don't dance-Well they're are no friends of mine. I say, we can go where we want to, a place where they will never find. And we can act like we come from out of this world Leave the real one far behind"
- board text added: "He is the Messiah!"
- board text added: "He who hesistates is sometimes saved"
- board text added: "Will you please listen? I am not the Messiah"
Changed lines of the file:
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@@
   (general
     (thickness 1.6)
-    (drawings 13)
+    (drawings 17)
     (tracks 145)
     (zones 0)
-    (modules 24)
+    (modules 25)
     (nets 14)
   )
   (page A4)
   (layers
-    (0 F.Cu signal)
-    (31 B.Cu power)
-    (32 B.Adhes user hide)
+    (0 F.Cu signal hide)
+    (31 B.Cu power hide)
+    (32 B.Adhes user)
     (33 F.Adhes user)
-    (34 B.Paste user hide)
+    (34 B.Paste user)
     (35 F.Paste user)
-    (36 B.SilkS user hide)
+    (36 B.SilkS user)
     (37 F.SilkS user)
-    (38 B.Mask user hide)
+    (38 B.Mask user)
     (39 F.Mask user)
     (40 Dwgs.User user)
@@
     (44 Edge.Cuts user)
     (45 Margin user)
-    (46 B.CrtYd user hide)
+    (46 B.CrtYd user)
     (47 F.CrtYd user)
     (48 B.Fab user hide)
@@
   )
   (module marion:caribiner-bsilks (layer F.Cu)
-    (at 188.341 77.597)
+    (at 188.341 78.74)
     (fp_text reference G*** (at -6.35 3.81) (layer F.SilkS) hide
       (effects (font (size 1.524 1.524) (thickness 0.3)))
@@
       (rotate (xyz 0 0 0))
     )
+  )
+  (module marion:avengers (layer F.Cu)
+    (at 201.93 79.248)
+    (fp_text reference G*** (at 0 0) (layer F.SilkS) hide
+      (effects (font (size 1.524 1.524) (thickness 0.3)))
+    )
+    (fp_text value LOGO (at 0.75 0) (layer F.SilkS) hide
+      (effects (font (size 1.524 1.524) (thickness 0.3)))
+    )
+    (fp_poly (pts (xy -2.03679 -2.034539) (xy -2.032751 -1.976091) (xy -2.032 -1.9304) (xy -2.032 -1.8034)
+      (xy -2.173817 -1.8034) (xy -2.249192 -1.8069) (xy -2.297184 -1.81595) (xy -2.307167 -1.825261)
+      (xy -2.285466 -1.850954) (xy -2.238069 -1.896581) (xy -2.177547 -1.951089) (xy -2.116469 -2.003428)
+      (xy -2.067403 -2.042544) (xy -2.043156 -2.0574) (xy -2.03679 -2.034539)) (layer F.SilkS) (width 0.01))
+    (fp_poly (pts (xy -2.172865 -3.677728) (xy -2.0193 -3.6703) (xy -2.011947 -3.462202) (xy -2.007591 -3.359528)
+      (xy -2.000231 -3.294649) (xy -1.985077 -3.254589) (xy -1.957344 -3.226373) (xy -1.91465 -3.198515)
+      (xy -1.814314 -3.116498) (xy -1.714543 -3.000209) (xy -1.627009 -2.864947) (xy -1.572158 -2.749603)
+      (xy -1.529963 -2.592704) (xy -1.512827 -2.41491) (xy -1.520884 -2.236072) (xy -1.554264 -2.076041)
+      (xy -1.567436 -2.039133) (xy -1.672626 -1.837553) (xy -1.812159 -1.669507) (xy -1.980902 -1.538568)
+      (xy -2.173724 -1.448312) (xy -2.385492 -1.402314) (xy -2.4892 -1.397) (xy -2.602664 -1.403994)
+      (xy -2.719823 -1.422617) (xy -2.825313 -1.449335) (xy -2.903769 -1.480613) (xy -2.929704 -1.498359)
+      (xy -2.933433 -1.531384) (xy -2.917149 -1.585634) (xy -2.887754 -1.639253) (xy -2.883422 -1.644922)
+      (xy -2.858748 -1.641127) (xy -2.802117 -1.623985) (xy -2.766213 -1.611622) (xy -2.625134 -1.579978)
+      (xy -2.462615 -1.572518) (xy -2.301887 -1.589232) (xy -2.212958 -1.611852) (xy -2.112318 -1.658533)
+      (xy -2.005722 -1.728838) (xy -1.957836 -1.768294) (xy -1.824443 -1.919708) (xy -1.733588 -2.090962)
+      (xy -1.685586 -2.274457) (xy -1.68075 -2.462596) (xy -1.719395 -2.647781) (xy -1.801834 -2.822412)
+      (xy -1.908618 -2.959005) (xy -2.030905 -3.0861) (xy -2.031453 -2.680568) (xy -2.032 -2.275036)
+      (xy -2.1717 -2.413) (xy -2.3114 -2.550965) (xy -2.312422 -2.831233) (xy -2.313444 -3.1115)
+      (xy -2.459796 -2.7686) (xy -2.513058 -2.643491) (xy -2.560076 -2.532462) (xy -2.59679 -2.445141)
+      (xy -2.619142 -2.391156) (xy -2.623077 -2.38125) (xy -2.62681 -2.357151) (xy -2.608259 -2.343715)
+      (xy -2.557573 -2.337938) (xy -2.47739 -2.3368) (xy -2.389174 -2.338088) (xy -2.339587 -2.345005)
+      (xy -2.316471 -2.362135) (xy -2.307664 -2.394059) (xy -2.306738 -2.401112) (xy -2.300938 -2.430284)
+      (xy -2.287884 -2.43958) (xy -2.259899 -2.42527) (xy -2.209308 -2.383618) (xy -2.136768 -2.318459)
+      (xy -1.974835 -2.171496) (xy -2.128272 -2.050948) (xy -2.203074 -1.993594) (xy -2.262002 -1.951041)
+      (xy -2.294261 -1.93102) (xy -2.296555 -1.9304) (xy -2.308558 -1.951791) (xy -2.3114 -1.982154)
+      (xy -2.314621 -2.00644) (xy -2.330703 -2.021157) (xy -2.369274 -2.028148) (xy -2.439962 -2.029256)
+      (xy -2.543605 -2.026604) (xy -2.77581 -2.0193) (xy -3.060046 -1.3716) (xy -3.244523 -1.3716)
+      (xy -3.333977 -1.373673) (xy -3.399529 -1.379142) (xy -3.428566 -1.386885) (xy -3.429 -1.388014)
+      (xy -3.418349 -1.412483) (xy -3.388325 -1.476624) (xy -3.341825 -1.574449) (xy -3.281747 -1.699971)
+      (xy -3.210987 -1.847203) (xy -3.132442 -2.010158) (xy -3.049008 -2.182848) (xy -2.963584 -2.359286)
+      (xy -2.879064 -2.533484) (xy -2.798347 -2.699456) (xy -2.724329 -2.851215) (xy -2.659907 -2.982773)
+      (xy -2.607978 -3.088142) (xy -2.571438 -3.161336) (xy -2.563001 -3.177892) (xy -2.555906 -3.201909)
+      (xy -2.575375 -3.209229) (xy -2.631471 -3.202047) (xy -2.654481 -3.197855) (xy -2.833925 -3.139124)
+      (xy -2.99593 -3.035697) (xy -3.134269 -2.892423) (xy -3.221859 -2.7559) (xy -3.254466 -2.688061)
+      (xy -3.274556 -2.624479) (xy -3.285048 -2.549181) (xy -3.288863 -2.44619) (xy -3.289178 -2.3876)
+      (xy -3.28637 -2.255501) (xy -3.276654 -2.161692) (xy -3.258329 -2.093928) (xy -3.244198 -2.06375)
+      (xy -3.216165 -2.004011) (xy -3.214952 -1.959497) (xy -3.2385 -1.905) (xy -3.270859 -1.853375)
+      (xy -3.29724 -1.829074) (xy -3.299184 -1.8288) (xy -3.319601 -1.850146) (xy -3.352941 -1.906194)
+      (xy -3.392099 -1.98496) (xy -3.393291 -1.98755) (xy -3.429039 -2.071996) (xy -3.450919 -2.146469)
+      (xy -3.462234 -2.228998) (xy -3.466289 -2.337607) (xy -3.46661 -2.3876) (xy -3.465216 -2.507224)
+      (xy -3.458103 -2.594166) (xy -3.441739 -2.666496) (xy -3.412592 -2.742285) (xy -3.385995 -2.800116)
+      (xy -3.272638 -2.987565) (xy -3.127915 -3.143777) (xy -2.95868 -3.263655) (xy -2.771785 -3.342106)
+      (xy -2.617831 -3.371289) (xy -2.470039 -3.38469) (xy -2.398235 -3.534923) (xy -2.32643 -3.685155)
+      (xy -2.172865 -3.677728)) (layer F.SilkS) (width 0.01))
+  )
+  (gr_text "He is the Messiah!" (at 208.8134 73.533 90) (layer F.SilkS)
+    (effects (font (size 0.0635 0.0635) (thickness 0.015875)))
+  )
+  (gr_text "Will you please listen? I am not the Messiah" (at 171.577 89.662) (layer F.SilkS)
+    (effects (font (size 0.0635 0.0635) (thickness 0.015875)))
+  )
+  (gr_text "Ah we can dance if we want to, we can leave your friends behind. Cause your friends don't dance and if they don't dance-Well they're are no friends of mine. \nI say, we can go where we want to, a place where they will never find. And we can act like we come from out of this world Leave the real one far behind" (at 184.4802 66.9798) (layer F.SilkS)
+    (effects (font (size 0.0635 0.0635) (thickness 0.015875)))
+  )
+  (gr_text "He who hesistates is sometimes saved" (at 183.134 72.5932 270) (layer B.Mask)
+    (effects (font (size 0.0635 0.0635) (thickness 0.015875)) (justify mirror))
   )
   (gr_line (start 211.328 88.392) (end 211.328 69.596) (layer Edge.Cuts) (width 0.15))
@@
     (polygon
       (pts
-        (xy 238.125 47.176577) (xy 115.57 47.176577) (xy 115.57 120.201577) (xy 241.3 120.201577) (xy 241.3 47.176577)
+        (xy 165.1 66.548) (xy 211.328 66.548) (xy 211.328 91.44) (xy 165.1 91.44)
       )
     )
