File: vreg-741.sch (KiCad schematic (older format))
At the start: 23 parts, among them J1 1729128, J2 1729128, Q1 FQT5P10, Q2 2STN1550, SW1 A6SN-1104, U1 UA741CDR‎

Commit message: extra easter eggs
Parts:
- D1: value 475-2486-1-ND -> 475-2486-1-ND
